Commit message: Update for new coordinate urdf and xml files

File: src/dyros_jet/dyros_jet_description/dyros_jet_robot_virtual.urdf (robot description, URDF)
Before this commit: robot dyros_jet_robot, 30 links, 29 joints
Joints:
- joint virtual: limit (none) -> lower=-3.14 upper=3.14 effort=30 velocity=1.0
